Commit message: modify urdf

File: office_world/urdf/office_robot.urdf (robot description, URDF)
Before this commit: robot IMRrobot, 9 links, 8 joints
Links:
- removed link base_link
- removed link imu_link
- removed link lidar_link
- removed link sensor_head_link
- removed link sonar0
- removed link sonar1
- removed link sonar2
- removed link sonar3
- removed link sonar4
- added link camera_link, mass 0.1; collision box size=0.05 0.05 0.05; visual box size=0.05 0.05 0.05
- added link camera_link_optical
- added link chassis, mass 15.0; collision box size=.42 .5 .1; visual box size=.42 .5 .1
- added link hokuyo, mass 1e-5; collision box size=0.1 0.1 0.1; visual mesh filename=package://my_robot/meshes/hokuyo.dae
- added link left_back_wheel, mass 5.0; collision cylinder length=0.05 radius=0.1; visual cylinder length=0.05 radius=0.1
- added link left_front_wheel, mass 5.0; collision cylinder length=0.05 radius=0.1; visual cylinder length=0.05 radius=0.1
- added link right_back_wheel, mass 5.0; collision cylinder length=0.05 radius=0.1; visual cylinder length=0.05 radius=0.1
- added link right_front_wheel, mass 5.0; collision cylinder length=0.05 radius=0.1; visual cylinder length=0.05 radius=0.1
- added link robot_footprint
Joints:
- removed joint imu_link_joint
- removed joint lidar_link_joint
- removed joint sensor_head_link_joint
- removed joint sonar0_joint
- removed joint sonar1_joint
- removed joint sonar2_joint
- removed joint sonar3_joint
- removed joint sonar4_joint
- added joint camera_joint: type fixed, parent chassis, child camera_link, origin xyz=0.21 0 0 rpy=0 0 0, axis 0 1 0
- added joint camera_optical_joint: type fixed, parent camera_link, child camera_link_optical, origin xyz=0 0 0 rpy=-1.5707 0 -1.5707
- added joint hokuyo_joint: type fixed, parent chassis, child hokuyo, origin xyz=0.21 0 0.1 rpy=0 0 0, axis 0 1 0
- added joint left_back_wheel_hinge: type continuous, parent chassis, child left_back_wheel, origin xyz=-0.11 0.3 0 rpy=0 0 0, axis 0 1 0, limit effort=10000 velocity=1000
- added joint left_front_wheel_hinge: type continuous, parent chassis, child left_front_wheel, origin xyz=0.11 0.3 0 rpy=0 0 0, axis 0 1 0, limit effort=10000 velocity=1000
- added joint right_back_wheel_hinge: type continuous, parent chassis, child right_back_wheel, origin xyz=-0.11 -0.3 0 rpy=0 0 0, axis 0 1 0, limit effort=10000 velocity=1000
- added joint right_front_wheel_hinge: type continuous, parent chassis, child right_front_wheel, origin xyz=0.11 -0.3 0 rpy=0 0 0, axis 0 1 0, limit effort=10000 velocity=1000
- added joint robot_footprint_joint: type fixed, parent robot_footprint, child chassis, origin xyz=0 0 0.1 rpy=0 0 0
